Commit message: Added spawn file for Gazebo

File: RoboCon2019/TestCodes/Quadruped/ROS-Aditya/robot_description/urdf/links_joints.xacro (robot description, xacro)
@@ -36,4 +36,9 @@
   <xacro:macro name="BOX" params="name origin_xyz origin_rpy size">
     <link name="${name}">
+       <inertial>
+        <mass value="10" />
+        <origin rpy="${origin_rpy}" xyz="${origin_xyz}" />
+        <inertia ixx="1" ixy="1" ixz="1" iyy="1" iyz="1" izz="1" />
+      </inertial>
       <collision>
         <origin rpy="${origin_rpy}" xyz="${origin_xyz}" />

Commit message: Added control for gazebo

File: RoboCon2019/TestCodes/Quadruped/ROS-Aditya/robot_description/urdf/links_joints.xacro (robot description, xacro)
@@ -9,4 +9,14 @@
       <child link="${child}" />
     </joint>
+    <transmission name="trans_${name}">
+      <type>transmission_interface/SimpleTransmission</type>
+      <joint name="${name}">
+        <hardwareInterface>hardware_interface/EffortJointInterface</hardwareInterface>
+      </joint>
+      <actuator name="motor_${name}">
+        <hardwareInterface>hardware_interface/EffortJointInterface</hardwareInterface>
+        <mechanicalReduction>1</mechanicalReduction>
+      </actuator>
+    </transmission>
   </xacro:macro>
   <xacro:macro name="JOINT_FIXED" params="name axis_xyz origin_rpy origin_xyz parent child ">

File: RoboCon2019/TestCodes/Quadruped/ROS-Aditya/robot_description/urdf/robot.xacro (robot description, xacro)
@@ -31,3 +31,7 @@
     <BOX name="link8" origin_rpy="0 0 0" origin_xyz="0 0 -0.475" size="0.3 0.48 0.95"/>
     <JOINT_REVOLUTE name="dxel4__link8" parent="dxel4" child="link8" origin_rpy="0 0 0" origin_xyz="-0.48855 0.16 -0.18" axis_xyz="0 1 0"/>
+    <gazebo>
+    <plugin name="gazebo_ros_control" filename="libgazebo_ros_control.so">
+    </plugin>
+  </gazebo>
 </robot>
