Commit message: Added yaml file

File: RoboCon2019/TestCodes/Quadruped/ROS-Ak/quadped1/urdf/links_joints.xacro (robot description, xacro)
@@ -9,4 +9,14 @@
       <child link="${child}" />
     </joint>
+    <transmission name="trans_${name}">
+      <type>transmission_interface/SimpleTransmission</type>
+      <joint name="${name}">
+        <hardwareInterface >hardware_interface/EffortJointInterface</hardwareInterface>
+      </joint>
+      <actuator name="motor_${name}">
+        <hardwareInterface>hardware_interface/EffortJointInterface</hardwareInterface>
+        <mechanicalReduction>1</mechanicalReduction>
+      </actuator>
+    </transmission>
   </xacro:macro>
   <xacro:macro name="JOINT_FIXED" params="name axis_xyz origin_rpy origin_xyz parent child ">

File: RoboCon2019/TestCodes/Quadruped/ROS-Ak/quadped1/urdf/robot.xacro (robot description, xacro)
@@ -1,4 +1,4 @@
 <?xml version="1.0" ?>
-<robot name="mrm" xmlns:xacro="http://www.ros.org/wiki/xacro">
+<robot name="robot" xmlns:xacro="http://www.ros.org/wiki/xacro">
     <xacro:include filename="$(find quadped1)/urdf/links_joints.xacro"/>
     <!--first leg -->
@@ -31,3 +31,7 @@
     <BOX name="link8" origin_rpy="0 0 0" origin_xyz="0 0 -0.475" size="0.3 0.48 0.95"/>
     <JOINT_REVOLUTE name="dxel4__link8" parent="dxel4" child="link8" origin_rpy="0 0 0" origin_xyz="-0.48855 0.16 -0.18" axis_xyz="0 1 0"/>
+    <gazebo>
+    <plugin name="gazebo_ros_control" filename="libgazebo_ros_control.so">
+    </plugin>
+  </gazebo>
 </robot>
