Commit message: robot_leg loop fix

File: RoboCon2019/TestCodes/Quadruped/ROS-Ak/robot_leg/urdf/links_joints.xacro (robot description, xacro)
@@ -83,5 +83,7 @@
           <mesh filename="${meshfile}" scale="${meshscale}"/>
         </geometry>
-        <material name="light_black"/>
+        <material name="silver">
+          <color rgba="${192/255} ${192/255} ${192/255} 1.0"/>
+        </material>
       </visual>
     </link>

File: RoboCon2019/TestCodes/Quadruped/ROS-Ak/robot_leg/urdf/robot.xacro (robot description, xacro)
@@ -6,5 +6,5 @@
           origin_xyz="0 0 0"
           origin_rpy="1.57070 0 0"
-	  meshfile="package://robot_leg/meshes/frame.stl"
+	  meshfile="package://robot_leg/meshes/frame.dae"
 	  meshscale="1 1 1"
 	  mass="1"
@@ -20,5 +20,5 @@
           origin_xyz="0 -0.2011 0.038"
           origin_rpy="1.57070 0 0"
-	  meshfile="package://new_robot/meshes/upper link right.stl"
+	  meshfile="package://new_robot/meshes/upper link right.dae"
 	  meshscale="1 1 1"
 	  mass="1"
@@ -34,5 +34,5 @@
           origin_xyz="0 0.012 0.1412"
           origin_rpy="1.57070 0 0"
-	  meshfile="package://new_robot/meshes/lower link right.stl"
+	  meshfile="package://new_robot/meshes/lower link right.dae"
 	  meshscale="1 1 1"
 	  mass="1"
@@ -48,5 +48,5 @@
           origin_xyz="0.25 -0.575 0.15"
           origin_rpy="1.9607 0 3.1416"
-	  meshfile="package://robot_leg/meshes/upper link left.stl"
+	  meshfile="package://robot_leg/meshes/upper link left.dae"
 	  meshscale="1 1 1"
 	  mass="1"
@@ -62,5 +62,5 @@
           origin_xyz="0.25 -0.42 0.09"
           origin_rpy="1.57070 0 3.1416"
-	  meshfile="package://robot_leg/meshes/lower link left.stl"
+	  meshfile="package://robot_leg/meshes/lower link left.dae"
 	  meshscale="1 1 1"
 	  mass="1"
@@ -77,5 +77,5 @@
           origin_xyz="0.25 -0.575 0.15"
           origin_rpy="1.9607 0 3.1416"
-	  meshfile="package://robot_leg/meshes/upper link left.stl"
+	  meshfile="package://robot_leg/meshes/upper link left.dae"
 	  meshscale="1 1 1"
 	  mass="1"
@@ -91,5 +91,5 @@
           origin_xyz="0.25 -0.42 0.09"
           origin_rpy="1.57070 0 3.1416"
-	  meshfile="package://new_robot/meshes/lower link left.stl"
+	  meshfile="package://new_robot/meshes/lower link left.dae"
 	  meshscale="1 1 1"
 	  mass="1"
@@ -105,5 +105,5 @@
           origin_xyz="0 -0.2011 0.038"
           origin_rpy="1.57070 0 0"
-	  meshfile="package://new_robot/meshes/upper link right.stl"
+	  meshfile="package://new_robot/meshes/upper link right.dae"
 	  meshscale="1 1 1"
 	  mass="1"
@@ -119,5 +119,5 @@
           origin_xyz="0 0.012 0.1412"
           origin_rpy="1.57070 0 0"
-	  meshfile="package://new_robot/meshes/lower link right.stl"
+	  meshfile="package://new_robot/meshes/lower link right.dae"
 	  meshscale="1 1 1"
 	  mass="1"
